Commit message: Update robot parameters

File: GoChaseIt/catkin_ws/src/my_robot/urdf/my_robot.xacro (robot description, xacro)
@@ -1,4 +1,18 @@
 <robot name="my_robot" xmlns:xacro="http://www.ros.org/wiki/xacro">
   <xacro:include filename="$(find my_robot)/urdf/my_robot.gazebo" />
+  <!-- Define materials -->
+  <xacro:macro name="material_orange">
+    <material name="orange">
+      <color rgba="0.929 0.6 0.196 1"/>
+    </material>
+  </xacro:macro>
+  <xacro:macro name="material_brown">
+    <material name="brown">
+      <color rgba="0.596 0.474 0.325 1"/>
+    </material>
+  </xacro:macro>
+  <!-- Use macros for materials -->
+  <xacro:material_orange/>
+  <xacro:material_brown/>
   <link name="robot_footprint"></link>
   <joint name="robot_footprint_joint" type="fixed">
@@ -10,5 +24,5 @@
     <pose>0 0 0.1 0 0 0</pose>
     <inertial>
-      <mass value="15.0"/>
+      <mass value="10.0"/>
       <origin xyz="0.0 0 0" rpy=" 0 0 0"/>
       <inertia
@@ -21,5 +35,5 @@
       <origin xyz="0 0 0" rpy=" 0 0 0"/>
       <geometry>
-        <box size=".4 .2 .1"/>
+        <box size=".4 .3 .1"/>
       </geometry>
     </collision>
@@ -27,11 +41,12 @@
       <origin xyz="0 0 0" rpy=" 0 0 0"/>
       <geometry>
-        <box size=".4 .2 .1"/>
+        <box size=".4 .3 .1"/>
       </geometry>
+      <material name="orange"/>
     </visual>
     <collision name='back_caster_collision'>
       <origin xyz="-0.15 0 -0.05" rpy=" 0 0 0"/>
       <geometry>
-        <sphere radius="0.0499"/>
+        <sphere radius="0.0599"/>
       </geometry>
     </collision>
@@ -39,5 +54,5 @@
       <origin xyz="-0.15 0 -0.05" rpy=" 0 0 0"/>
       <geometry>
-        <sphere radius="0.05"/>
+        <sphere radius="0.06"/>
       </geometry>
     </visual>
@@ -45,5 +60,5 @@
       <origin xyz="0.15 0 -0.05" rpy=" 0 0 0"/>
       <geometry>
-        <sphere radius="0.0499"/>
+        <sphere radius="0.0599"/>
       </geometry>
     </collision>
@@ -51,5 +66,5 @@
       <origin xyz="0.15 0 -0.05" rpy=" 0 0 0"/>
       <geometry>
-        <sphere radius="0.05"/>
+        <sphere radius="0.06"/>
       </geometry>
     </visual>
@@ -65,5 +80,5 @@
       <origin rpy="0 1.5707 1.5707" xyz="0 0 0" />
       <geometry>
-        <cylinder radius="0.1" length="0.05" />
+        <cylinder radius="0.12" length="0.05" />
       </geometry>
     </collision>
@@ -71,10 +86,11 @@
       <origin rpy="0 1.5707 1.5707" xyz="0 0 0" />
       <geometry>
-        <cylinder radius="0.1" length="0.05" />
+        <cylinder radius="0.12" length="0.05" />
       </geometry>
+      <material name="brown"/>
     </visual>
   </link>
   <joint name="left_wheel_hinge" type="continuous">
-    <origin rpy="0 0 0" xyz="0 0.15 0" />
+    <origin rpy="0 0 0" xyz="0 0.18 0" />
     <parent link="chassis" />
     <child link="left_wheel" />
@@ -93,5 +109,5 @@
       <origin rpy="0 1.5707 1.5707" xyz="0 0 0" />
       <geometry>
-        <cylinder radius="0.1" length="0.05" />
+        <cylinder radius="0.12" length="0.05" />
       </geometry>
     </collision>
@@ -99,10 +115,11 @@
       <origin rpy="0 1.5707 1.5707" xyz="0 0 0" />
       <geometry>
-        <cylinder radius="0.1" length="0.05" />
+        <cylinder radius="0.12" length="0.05" />
       </geometry>
+      <material name="brown"/>
     </visual>
   </link>
   <joint name="right_wheel_hinge" type="continuous">
-    <origin rpy="0 0 0" xyz="0 -0.15 0" />
+    <origin rpy="0 0 0" xyz="0 -0.18 0" />
     <parent link="chassis" />
     <child link="right_wheel" />

Commit message: Fix world and robot stability

File: GoChaseIt/catkin_ws/src/my_robot/urdf/my_robot.xacro (robot description, xacro)
@@ -46,5 +46,5 @@
     </visual>
     <collision name='back_caster_collision'>
-      <origin xyz="-0.15 0 -0.05" rpy=" 0 0 0"/>
+      <origin xyz="-0.15 0 -0.06" rpy=" 0 0 0"/>
       <geometry>
         <sphere radius="0.0599"/>
@@ -52,5 +52,5 @@
     </collision>
     <visual name='back_caster_visual'>
-      <origin xyz="-0.15 0 -0.05" rpy=" 0 0 0"/>
+      <origin xyz="-0.15 0 -0.06" rpy=" 0 0 0"/>
       <geometry>
         <sphere radius="0.06"/>
@@ -58,5 +58,5 @@
     </visual>
     <collision name='front_caster_collision'>
-      <origin xyz="0.15 0 -0.05" rpy=" 0 0 0"/>
+      <origin xyz="0.15 0 -0.06" rpy=" 0 0 0"/>
       <geometry>
         <sphere radius="0.0599"/>
@@ -64,5 +64,5 @@
     </collision>
     <visual name='front_caster_visual'>
-      <origin xyz="0.15 0 -0.05" rpy=" 0 0 0"/>
+      <origin xyz="0.15 0 -0.06" rpy=" 0 0 0"/>
       <geometry>
         <sphere radius="0.06"/>

Commit message: Fix process image code and colors

File: GoChaseIt/catkin_ws/src/my_robot/urdf/my_robot.xacro (robot description, xacro)
@@ -70,4 +70,7 @@
     </visual>
   </link>
+  <gazebo reference="chassis">
+    <material>Gazebo/Yellow</material>
+  </gazebo>
   <!-- Left Wheel -->
   <link name="left_wheel">
@@ -91,4 +94,7 @@
     </visual>
   </link>
+  <gazebo reference="left_wheel">
+    <material>Gazebo/Red</material>
+  </gazebo>
   <joint name="left_wheel_hinge" type="continuous">
     <origin rpy="0 0 0" xyz="0 0.18 0" />
@@ -120,4 +126,7 @@
     </visual>
   </link>
+  <gazebo reference="right_wheel">
+    <material>Gazebo/Red</material>
+  </gazebo>
   <joint name="right_wheel_hinge" type="continuous">
     <origin rpy="0 0 0" xyz="0 -0.18 0" />
@@ -148,4 +157,7 @@
     </visual>
   </link>
+  <gazebo reference="camera">
+    <material>Gazebo/Green</material>
+  </gazebo>
   <joint name="camera_joint" type="fixed">
     <origin rpy="0 0 0" xyz="0.2 0 0" />
