Commit message: Added mapping.launch file

File: MapMyWorld/catkin_ws/src/my_robot/urdf/my_robot.xacro (robot description, xacro)
@@ -192,3 +192,11 @@
     <axis xyz="0 1 0" />
   </joint>
+  <!-- Optical camera -->
+  <joint name="camera_optical_joint" type="fixed">
+    <origin xyz="0 0 0" rpy="-1.5707 0 -1.5707"/>
+    <parent link="camera"/>
+    <child link="camera_link_optical"/>
+  </joint>
+  <link name="camera_link_optical">
+  </link>
 </robot>

Commit message: Change rotation and add map db

File: MapMyWorld/catkin_ws/src/my_robot/urdf/my_robot.xacro (robot description, xacro)
@@ -194,5 +194,5 @@
   <!-- Optical camera -->
   <joint name="camera_optical_joint" type="fixed">
-    <origin xyz="0 0 0" rpy="-1.5707 0 -1.5707"/>
+    <origin xyz="0 0 0" rpy="0 0 -1.5707"/>
     <parent link="camera"/>
     <child link="camera_link_optical"/>

Commit message: Added teleop, updated mapping and fix camera orientation and added link to databast

File: MapMyWorld/catkin_ws/src/my_robot/urdf/my_robot.xacro (robot description, xacro)
@@ -194,5 +194,5 @@
   <!-- Optical camera -->
   <joint name="camera_optical_joint" type="fixed">
-    <origin xyz="0 0 0" rpy="0 0 -1.5707"/>
+    <origin xyz="0 0 0" rpy="-1.5707 0 -1.5707"/>
     <parent link="camera"/>
     <child link="camera_link_optical"/>
